Commit message: added battery, began to look into adding collisions and inertia values

File: src/my_robot_bringup/urdf/my_robot.urdf (robot description, URDF)
Before this commit: robot honors_thesis, 7 links, 6 joints
Links:
- added link battery; visual box size=0.178 0.203 0.14
- link base_link: geometry visual box size=0.4445 0.4318 0.05
- link lidar: geometry visual cylinder length=0.05 radius=.05
Joints:
- added joint base_battery_joint: type fixed, parent base_link, child battery, origin xyz=-0.111125 0 0 rpy=0 0 0
- joint base_lidar_joint: origin xyz=0 0 0.175 rpy=0 0 0 -> xyz=0.111125 0 0.05 rpy=0 0 0

Commit message: created all inertia and mass values based off of physical specs + added gazebo plugin

File: src/my_robot_bringup/urdf/my_robot.urdf (robot description, URDF)
Before this commit: robot honors_thesis, 8 links, 7 joints
Links:
- link back_left_wheel: mass None -> 0.8; geometry collision cylinder length=0.05 radius=0.089; visual cylinder length=0.05 radius=0.089
- link back_right_wheel: mass None -> 0.8; geometry collision cylinder length=0.05 radius=0.089; visual cylinder length=0.05 radius=0.089
- link base_link: mass None -> 13.6; geometry collision box size=0.4445 0.4318 0.05; visual box size=0.4445 0.4318 0.05
- link battery: mass None -> 5.44; geometry collision box size=0.178 0.203 0.14; visual box size=0.178 0.203 0.14
- link front_left_wheel: mass None -> 0.8; geometry collision cylinder length=0.05 radius=0.089; visual cylinder length=0.05 radius=0.089
- link front_right_wheel: mass None -> 0.8; geometry collision cylinder length=0.05 radius=0.089; visual cylinder length=0.05 radius=0.089
- link lidar: mass None -> 0.001; geometry collision cylinder length=0.05 radius=.05; visual cylinder length=0.05 radius=.05

Commit message: mostly resolved slam mapping issue with map not correctly populating

File: src/my_robot_bringup/urdf/my_robot.urdf (robot description, URDF)
Before this commit: robot honors_thesis, 8 links, 7 joints
Joints:
- joint base_lidar_joint: origin xyz=0.111125 0 0.05 rpy=0 0 0 -> xyz=0.111125 0 0.15 rpy=0 0 0
